File: arquivoProjeto.brd (EAGLE design)
At the start: 261 x 78.3 mm, 12 parts, among them U1 ARDUINO-UNO-R3-SHIELD, U2 LCD-16X2JHD-162A

Commit message: refactor: Atualização de .BRD
Parts:
- moved PIEZO1 58.7 mm to (208.1, 107.4), turned to -90 degrees
- moved R6 53.8 mm to (167.3, 59.4)
- moved R5 53.8 mm to (160.9, 64.4)
- moved D1 12.7 mm to (194.0, 54.3), turned to 180 degrees
- moved D2 12.7 mm to (219.4, 54.3), turned to 180 degrees
- moved D3 12.7 mm to (242.2, 54.3), turned to 180 degrees
- turned R2 to 0 degrees
- turned R3 to 0 degrees
- turned R4 to 0 degrees
Other:
- board size 261 x 78.3 mm -> 257.5 x 119.2 mm
